Commit message: URDF changed and bringup launch file added for the GoPiGo3 instance at BME AUT

File: gopigo3_description/urdf/gopigo3.urdf.xacro (robot description, xacro)
@@ -216,5 +216,5 @@
       <parent link="base_link"/>
       <child link="base_scan"/>
-      <origin xyz="-0.02 0 0.085" rpy="0 0 -1.57"/>
+      <origin xyz="0 0 0.085" rpy="0 0 -3.1416"/>
       <!--LDS** origin xyz="-0.02 0 0.07" rpy="0 0 -1.6"/-->
     </joint>
