Commit message: New URDF added for the GoPiGo3 instance at BME AUT

File: gopigo3_description/urdf/gopigo3_bmeaut.urdf.xacro (robot description, xacro)
@@ -2,11 +2,11 @@
 <robot name="gopigo3" xmlns:xacro="http://ros.org/wiki/xacro">
   <xacro:include filename="$(find gopigo3_description)/urdf/common_properties.xacro"/>
-  <xacro:include filename="$(find gopigo3_description)/urdf/gopigo3.gazebo.xacro"/>
+  <xacro:include filename="$(find gopigo3_description)/urdf/gopigo3_bmeaut.gazebo.xacro"/>
   <xacro:property name="CADscale" value="0.0012" />
   <!-- Which sensors to include -->
 <xacro:arg name="imu" default="false" />
 <!--xacro:property name="imu" value="true"/-->
-<xacro:arg name="distance"        default="true"/>
-<xacro:arg name="pi_camera"       default="true"/>
+<xacro:arg name="distance"        default="false"/>
+<xacro:arg name="pi_camera"       default="false"/>
 <xacro:arg name="lds"             default="true"/>
 <!-- ============ 'base_footprint' is the ground link ===================== -->
@@ -164,5 +164,5 @@
   </link>
 <!-- ============ imu_link xacro:macro ========================= -->
-  <xacro:macro name="imu_sensor">
+  <!-- <xacro:macro name="imu_sensor">
     <joint name="imu_joint" type="fixed">
       <parent link="base_link"/>
@@ -179,5 +179,5 @@
       </visual>
     </link>
-  </xacro:macro>
+  </xacro:macro> -->
 <!-- ============ imu_link xacro:if ========================= -->
   <!-- if using a property (just inside this URDF file)-->
@@ -185,18 +185,18 @@
   <!--xacro:if value="${imu}"-->
   <!-- if using an argument (call from outside)-->
-  <xacro:if value="$(arg imu)">
+  <!-- <xacro:if value="$(arg imu)">
     <xacro:imu_sensor/>
-  </xacro:if>
+  </xacro:if> -->
 <!-- ============ Distance sensor ====================== -->
-  <xacro:macro name="distance_sensor">
+  <!-- <xacro:macro name="distance_sensor"> -->
   <!-- JOINT distance_sensor to base_link -->
-    <joint name="distance_sensor_joint" type="fixed">
+    <!-- <joint name="distance_sensor_joint" type="fixed">
       <axis xyz="0 1 0" />
       <origin xyz="0.065 0 0.025" rpy="0 0 0"/>
       <parent link="base_link"/>
       <child link="distance_sensor"/>
-    </joint>
+    </joint> -->
   <!-- Distance Sensor -->
-    <link name="distance_sensor">
+    <!-- <link name="distance_sensor">
       <visual>
         <origin xyz="0 0 0" rpy="1.57 0 1.57"/>
@@ -210,5 +210,5 @@
   <xacro:if value="$(arg distance)">
     <xacro:distance_sensor/>
-  </xacro:if>
+  </xacro:if> -->
 <!-- ============ base_scan ======================== -->
   <xacro:macro name="lds_sensor">
@@ -216,5 +216,5 @@
       <parent link="base_link"/>
       <child link="base_scan"/>
-      <origin xyz="-0.02 0 0.085" rpy="0 0 -1.57"/>
+      <origin xyz="0 0 0.085" rpy="0 0 -3.1416"/>
       <!--LDS** origin xyz="-0.02 0 0.07" rpy="0 0 -1.6"/-->
     </joint>
@@ -252,7 +252,7 @@
   </xacro:if>
 <!-- ============ Pi Camera ====================== -->
-  <xacro:macro name="pi_camera_sensor">
+  <!-- <xacro:macro name="pi_camera_sensor"> -->
   <!-- (LINKS) Pi Camera -->
-    <link name="camera_link">
+    <!-- <link name="camera_link">
       <visual>
         <origin xyz="0.005 0.000 0.013" rpy="0 1.570795 0" />
@@ -261,7 +261,7 @@
         </geometry>
         <material name="yellow"/>
-      </visual>
+      </visual> -->
     <!-- **** Pi Camera COLLISION & INERTIA **** -->
-      <collision>
+      <!-- <collision>
         <origin xyz="0.005 0 0.013" rpy="0 0 0"/>
         <geometry>
@@ -271,7 +271,7 @@
       </link>
     <link name="camera_rgb_frame"/>
-    <link name="camera_rgb_optical_frame"/>
+    <link name="camera_rgb_optical_frame"/> -->
   <!-- (JOINTS) Pi Camera -->
-    <joint name="camera_joint" type="fixed">
+    <!-- <joint name="camera_joint" type="fixed">
       <origin xyz="0.04 0 0.04" rpy="0 0 0"/>
       <parent link="base_link"/>
@@ -291,4 +291,4 @@
   <xacro:if value="$(arg pi_camera)">
     <xacro:pi_camera_sensor/>
-  </xacro:if>
+  </xacro:if> -->
 </robot>

Commit message: URDF changes to modify TF tree

File: gopigo3_description/urdf/gopigo3_bmeaut.urdf.xacro (robot description, xacro)
@@ -47,8 +47,8 @@
 <!-- ============  'base_link_cad' is the solid model of robot body ====== -->
   <joint name="base_joint_cad" type="fixed">
-    <parent link="base_footprint"/>
+    <parent link="base_link"/>
     <child link="base_link_cad"/>
     <!-- CAD of body of GoPiGo3 has its reference coordinate system at the center of the wheels shaft -->
-    <origin xyz="-0.02 0 0.033" rpy="0 0 -4.71"/>
+    <origin xyz="-0.02 0 -0.042" rpy="0 0 -4.71"/>
   </joint>
   <link name="base_link_cad">
